File: bldc_driver.kicad_sch (KiCad schematic)
At the start: 71 parts, among them J1 Conn_01x01_Pin, J10 Conn_01x01_Pin, J11 Conn_01x01_Pin, J2 USB_C_Receptacle_USB2.0_16P, J3 Conn_01x08_Pin, J4 Conn_ARM_SWD_TagConnect_TC203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, J5 Conn_01x03_Pin, J6 Conn_01x03_Pin, J7 Conn_01x03_Pin, J8 Conn_01x01_Pin, J9 Conn_01x01_Pin, SW1 SW_Push, U1 UA78M33QDCYRQ1, U2 SN65HVD230, U3 TPD2E2U06DCK, U4 AS5048A, U5 STM32G0B1KCTx, U6 DRV8317HREER, U7 AS5047D

Commit message: schematic and layout mostly done
Parts:
- removed C13: 10u, Capacitor_SMD:C_0603_1608Metric_Pad1.08x0.95mm_HandSolder, symbol Device:C
- removed J3: Conn_01x08_Pin, Connector_PinHeader_2.54mm:PinHeader_2x04_P2.54mm_Vertical, symbol Connector:Conn_01x08_Pin
- removed JP2: SolderJumper_2_Open, Jumper:SolderJumper-2_P1.3mm_Open_TrianglePad1.0x1.5mm, symbol Jumper:SolderJumper_2_Open
- removed U4: AS5048A, Package_SO:TSSOP-14_4.4x5mm_P0.65mm, symbol Sensor_Magnetic:AS5048A
- added J3: Conn_01x03_Pin, Connector_PinSocket_2.54mm:PinSocket_1x03_P2.54mm_Vertical, symbol Connector:Conn_01x03_Pin
- added R10, R11: 1k, Resistor_SMD:R_0402_1005Metric_Pad0.72x0.64mm_HandSolder, symbol Device:R
- added R12: 100k, Resistor_SMD:R_0402_1005Metric_Pad0.72x0.64mm_HandSolder, symbol Device:R
- added Y1: SiT8008xx-1x-xxE, Oscillator:Oscillator_SMD_SiT_PQFN-4Pin_2.5x2.0mm, symbol Oscillator:SiT8008xx-1x-xxE
- J2: footprint Connector_USB:USB_C_Receptacle_GCT_USB4110 -> bldc_driver:USB_C_Receptacle_GCT_USB4110
- U6: footprint WQFN36_REE_TEX -> bldc_driver:WQFN36_REE_TEX
Connections:
- net PA3 is gone; now on net nFAULT: U5.10 (PA3)
- net PB7 is gone; now on net ~{CAN_EN}: U5.31 (PB7)
- net PC6 is gone; now on net STATUS: U5.20 (PC6)
- net 3V3: now also C12.1, R_nFault1.1, R_nSLEEP1.2, U7.11 (VDD), U7.12 (VDD3V3), Y1.4 (Vdd)
- net AVDD_3V3: no longer R_nFault1.1, R_nSLEEP1.2
- net GND: now also U7.13 (GND), U7.5 (TST), J3.1 (Pin_1), R11.2, Y1.2 (GND)
- net PB2: now also U5.17 (PB2), J3.3 (Pin_3)
- net PB4: now also U5.28 (PB4), J3.2 (Pin_2)
- net SPI_CLK: now also U7.2 (CLK)
- net SPI_MISO: now also U7.3 (MISO)
- net SPI_MOSI: now also U7.4 (MOSI)
- net SPI_NSS: now also U7.1 (~{CS})
- net STATUS: now also R6.2; no longer R6.1, U5.2 (PC14)
- net VIN: now also R12.1
- net nRST: now also J4.3 (~{RESET})
- net ~{CAN_EN}: no longer U5.3 (PC15)
- net at D4.2 (A): now also R6.1; no longer R6.2
- net PA15 renamed VIN_SENS
- net VIN_SENS: now also R11.1, R12.2
- net USB_DM renamed USB_D-
- net USB_DP renamed USB_D+
- new net: U5.2 (PC14), Y1.3 (OUT)
- new net: R10.2, U5.3 (PC15)
- new net: R10.1, Y1.1 (OE)
- no-connect marks 9 -> 11
Other:
- note added: "CAN"
- note added: "Encoder"
- note added: "GPIO"
- note added: "Microcontroller"
- note added: "Motor Driver"
- note added: "Mounting"
- note added: "Power"
- note added: "USART"
- note added: "USB"
- company: (none) -> a-osb
- title: (none) -> bldc_driver
- moved on the sheet: C1, C10, C11, C12, C14, C15, C16, C17, C2, C3, C4, C5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

Commit message: for review with outputs
Parts:
- removed JP3, JP4: SolderJumper_2_Open, Jumper:SolderJumper-2_P1.3mm_Open_TrianglePad1.0x1.5mm, symbol Jumper:SolderJumper_2_Open
- removed R10: 1k, Resistor_SMD:R_0402_1005Metric_Pad0.72x0.64mm_HandSolder, symbol Device:R
- removed Y1: SiT8008xx-1x-xxE, Oscillator:Oscillator_SMD_SiT_PQFN-4Pin_2.5x2.0mm, symbol Oscillator:SiT8008xx-1x-xxE
- added Y1: ECS-2520MV-160-CN, bldc_driver:Oscillator_SMD_ECS_2520MV-xxx-xx-4Pin_2.5x2.0mm, symbol Oscillator:ECS-2520MV-xxx-xx
- C11: footprint Capacitor_SMD:C_0603_1608Metric_Pad1.08x0.95mm_HandSolder -> Capacitor_SMD:C_0402_1005Metric_Pad0.74x0.62mm_HandSolder
- C_CP1: Rating (none) -> 16V
- C_CSAREF1: value 0.1u -> 100n; Rating (none) -> 6.3V
- C_FLY1, C_VIN_AVDD1, C_VM1: value 0.1u -> 100n
- J1, J10, J11, J8, J9: now left out of the parts list
- J3, J6, J7: footprint Connector_PinSocket_2.54mm:PinSocket_1x03_P2.54mm_Vertical -> Connector_PinHeader_2.54mm:PinHeader_1x03_P2.54mm_Vertical; now not fitted; now left out of the parts list
- J5: now not fitted; now left out of the parts list
- R1: value 10k -> 5.1k
- R11: value 1k -> 5.1k
- R4: value 10K -> 5.1k
- R7, R8, R9: value 100R -> 120R
- R_term1: footprint Resistor_SMD:R_0201_0603Metric_Pad0.64x0.40mm_HandSolder -> Resistor_SMD:R_0402_1005Metric_Pad0.72x0.64mm_HandSolder
- U1: value UA78M33QDCYRQ1 -> UA78M33QDCYRG4Q1
Connections:
- net 3V3: now also Y1.4 (VDD)
- net GND: now also Y1.2 (GND)
- net USART_RX: now also U5.21 (PA10/UCPD1_DBCC2)
- net USART_TX: now also U5.19 (PA9/UCPD1_DBCC1)
- net CLK_16MHz: now reaches U5.2 (PC14)
- net CLK_16MHz: now also Y1.3 (OUT)
- no-connect marks 11 -> 13

Commit message: BOM with ratings
Parts:
- C1, C2, C3, C4, C5, C6, C8, C_VIN_AVDD1, C_VIN_AVDD2, C_VM1, C_VM2: Rating (none) -> 50V
- C11, C12, C14, C15, C16, C17, C7, C_AVDD1: Rating (none) -> 6.3V
Changed lines of the file:
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@@
 			)
 		)
+		(property "Rating" "6.3V"
+			(at 176.53 59.69 0)
+			(effects
+				(font
+					(size 1.27 1.27)
+				)
+				(hide yes)
+			)
+		)
 		(pin "1"
 		)
@@
 			)
 		)
+		(property "Rating" "50V"
+			(at 50.8 64.77 0)
+			(effects
+				(font
+					(size 1.27 1.27)
+				)
+				(hide yes)
+			)
+		)
 		(pin "2"
 		)
@@
 			)
 		)
+		(property "Rating" "6.3V"
+			(at 57.15 205.74 0)
+			(effects
+				(font
+					(size 1.27 1.27)
+				)
+				(hide yes)
+			)
+		)
 		(pin "1"
 		)
@@
 			)
 		)
+		(property "Rating" "50V"
+			(at 66.04 64.77 0)
+			(effects
+				(font
+					(size 1.27 1.27)
+				)
+				(hide yes)
+			)
+		)
 		(pin "2"
 		)
@@
 			)
 		)
+		(property "Rating" "50V"
+			(at 152.4 158.75 90)
+			(effects
+				(font
+					(size 1.27 1.27)
+				)
+				(hide yes)
+			)
+		)
 		(pin "2"
 		)
@@
 			)
 		)
+		(property "Rating" "50V"
+			(at 165.1 158.75 90)
+			(effects
+				(font
+					(size 1.27 1.27)
+				)
+				(hide yes)
+			)
+		)
 		(pin "1"
 		)
@@
 			)
 		)
+		(property "Rating" "6.3V"
+			(at 200.66 53.34 0)
+			(effects
+				(font
+					(size 1.27 1.27)
+				)
+				(hide yes)
+			)
+		)
 		(pin "2"
 		)
@@
 			)
 		)
+		(property "Rating" "6.3V"
+			(at 53.34 167.64 90)
+			(effects
+				(font
+					(size 1.27 1.27)
+				)
+				(hide yes)
+			)
+		)
 		(pin "1"
 		)
@@
 			)
 		)
+		(property "Rating" "50V"
+			(at 76.2 64.77 0)
+			(effects
+				(font
+					(size 1.27 1.27)
+				)
+				(hide yes)
+			)
+		)
 		(pin "2"
 		)
@@
 			)
 		)
+		(property "Rating" "50V"
+			(at 71.12 64.77 0)
+			(effects
+				(font
+					(size 1.27 1.27)
+				)
+				(hide yes)
+			)
+		)
 		(pin "2"
 		)
@@
 			)
 		)
+		(property "Rating" "6.3V"
+			(at 285.75 67.31 0)
+			(effects
+				(font
+					(size 1.27 1.27)
+				)
+				(hide yes)
+			)
+		)
 		(pin "1"
 		)
@@
 			)
 		)
+		(property "Rating" "50V"
+			(at 146.05 158.75 90)
+			(effects
+				(font
+					(size 1.27 1.27)
+				)
+				(hide yes)
+			)
+		)
 		(pin "2"
 		)
@@
 			)
 		)
+		(property "Rating" "6.3V"
+			(at 50.8 205.74 0)
+			(effects
+				(font
+					(size 1.27 1.27)
+				)
+				(hide yes)
+			)
+		)
 		(pin "1"
 		)
@@
 			)
 		)
+		(property "Rating" "50V"
+			(at 55.88 64.77 0)
+			(effects
+				(font
+					(size 1.27 1.27)
+				)
+				(hide yes)
+			)
+		)
 		(pin "2"
 		)
@@
 			)
 		)
+		(property "Rating" "6.3V"
+			(at 63.5 205.74 0)
+			(effects
+				(font
+					(size 1.27 1.27)
+				)
+				(hide yes)
+			)
+		)
 		(pin "1"
 		)
@@
 			)
 		)
+		(property "Rating" "50V"
+			(at 67.31 101.6 0)
+			(effects
+				(font
+					(size 1.27 1.27)
+				)
+				(hide yes)
+			)
+		)
 		(pin "2"
 		)
@@
 			)
 		)
+		(property "Rating" "50V"
+			(at 60.96 64.77 0)
+			(effects
+				(font
+					(size 1.27 1.27)
+				)
+				(hide yes)
+			)
+		)
 		(pin "2"
 		)
@@
 			)
 		)
+		(property "Rating" "6.3V"
+			(at 228.6 170.18 0)
+			(effects
+				(font
+					(size 1.27 1.27)
+				)
+				(hide yes)
+			)
+		)
 		(pin "1"
 		)
@@
 			(effects
 				(font
+					(size 1.27 1.27)
+				)
+				(hide yes)
+			)
+		)
+		(property "Rating" "50V"
+			(at 158.75 158.75 90)
+			(effects
+				(font

Commit message: cut rev 0.1
Parts:
- C_VIN_AVDD2, C_VM2: footprint Capacitor_SMD:C_0603_1608Metric_Pad1.08x0.95mm_HandSolder -> Capacitor_SMD:C_0805_2012Metric_Pad1.18x1.45mm_HandSolder
- SW1: footprint Button_Switch_SMD:SW_Tactile_SPST_NO_Straight_CK_PTS636Sx25SMTRLFS -> Button_Switch_SMD:SW_Push_1P1T_NO_CK_KMR2
Connections:
- net PB2: now also J3.2 (Pin_2); no longer J3.3 (Pin_3)
- net PB4: now also J3.3 (Pin_3); no longer J3.2 (Pin_2)
Changed lines of the file:
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@@
 		)
 	)
-	(text_box "TODO\n- horizontal push button for boot/reset\n- Test pads: 3v3, Vin, Encoder PWM, nRST, Boot0\n- Board shape\n\nDONE\n- Vsens voltage divider\n- switch to buck converter (instead of LDO) if low cost - won't do\n- Upgrade AS5048 to AS5047\n- Separate AGND from PGND in DRV8317? (as per user guide)\n- CAN connector, UART connector\n- bulk capacitance\n- ESD - TVS diodes - 5V or 3v3 for USB lines?\n- Boot0 to Gnd\n- Push button for reset\n- Status LEDs\n- Programming header\n- CAN transeiver from datasheet, has layout guide: https://www.ti.com/lit/ds/symlink/sn65hvd230.pdf\n- Encoder from datasheet\n- Decoupling capacitors"
-		(exclude_from_sim no)
-		(at 22.86 -50.8 0)
-		(size 73.66 45.72)
-		(margins 0.9525 0.9525 0.9525 0.9525)
-		(stroke
-			(width 0)
-			(type solid)
-		)
-		(fill
-			(type none)
-		)
-		(effects
-			(font
-				(size 1.27 1.27)
-			)
-			(justify left top)
-		)
-	)
-	(text_box "Notes:\n- C_VM2 - okay to use ceramic instead of electrolytic?\n- C_AVDD value chosen for no external load\n- Connect PGND to seperate ground plane\n"
-		(exclude_from_sim no)
-		(at -33.02 133.35 0)
-		(size 31.75 22.86)
-		(margins 0.9525 0.9525 0.9525 0.9525)
-		(stroke
-			(width 0)
-			(type solid)
-		)
-		(fill
-			(type none)
-		)
-		(effects
-			(font
-				(size 1.27 1.27)
-			)
-			(justify left top)
-		)
-	)
 	(text_box "Only connect R_term if the device is at the end of the bus"
 		(exclude_from_sim no)
@@
 	)
 	(image
-		(at 157.48 -29.21)
+		(at 187.96 -30.48)
 		(scale 1.11103)
 		(data "iVBORw0KGgoAAAANSUhEUgAAAooAAAJrCAIAAADoDiX8AAAAA3NCSVQICAjb4U/gAAAgAElEQVR4"
@@
 	)
 	(image
-		(at 466.09 99.06)
+		(at 233.68 308.61)
 		(data "iVBORw0KGgoAAAANSUhEUgAAA/sAAADhCAIAAAAYvzINAAAAA3NCSVQICAjb4U/gAAAgAElEQVR4"
 			"nOzdf1wTZ9ov/msIMhGaIDZRbAzWCBQQBAuiaxb3McoeAfcUsV+MdhV9qugWxbMiLrVwil+peqTY"
@@
 		)
 	)
-	(global_label "PB2"
-		(shape bidirectional)
-		(at 375.92 193.04 0)
-		(fields_autoplaced yes)
-		(effects
-			(font
-				(size 1.27 1.27)
-			)
-			(justify left)
-		)
-		(property "Intersheetrefs" "${INTERSHEET_REFS}"
-			(at 383.766 193.04 0)
-			(effects
-				(font
-					(size 1.27 1.27)
-				)
-				(justify left)
-				(hide yes)
-			)
-		)
-	)
 	(global_label "USART_RX"
 		(shape input)
@@
 		)
 	)
+	(global_label "PB2"
+		(shape bidirectional)
+		(at 375.92 195.58 0)
+		(fields_autoplaced yes)
+		(effects
+			(font
+				(size 1.27 1.27)
+			)
+			(justify left)
+		)
+		(property "Intersheetrefs" "${INTERSHEET_REFS}"
+			(at 383.766 195.58 0)
+			(effects
+				(font
+					(size 1.27 1.27)
+				)
+				(justify left)
+				(hide yes)
+			)
+		)
+	)
 	(global_label "CURR_SENS_B"
 		(shape input)
@@
 		)
 	)
-	(global_label "USB_D-"
+	(global_label "PB4"
 		(shape bidirectional)
-		(at 245.11 92.71 0)
+		(at 375.92 193.04 0)
 		(fields_autoplaced yes)
 		(effects
@@
 		)
 		(property "Intersheetrefs" "${INTERSHEET_REFS}"
-			(at 256.8265 92.71 0)
+			(at 383.766 193.04 0)
 			(effects
 				(font
@@
 		)
 	)
-	(global_label "SPI_NSS"
-		(shape output)
-		(at 220.98 186.69 180)
+	(global_label "USB_D-"
+		(shape bidirectional)
+		(at 245.11 92.71 0)
 		(fields_autoplaced yes)
 		(effects
@@
 				(size 1.27 1.27)
 			)
-			(justify right)
+			(justify left)
 		)
 		(property "Intersheetrefs" "${INTERSHEET_REFS}"
-			(at 210.1934 186.69 0)
+			(at 256.8265 92.71 0)
 			(effects
 				(font
 					(size 1.27 1.27)
 				)
-				(justify right)
+				(justify left)
 				(hide yes)
 			)
 		)
 	)
-	(global_label "3V3"
-		(shape input)
-		(at 144.78 67.31 180)
+	(global_label "SPI_NSS"
+		(shape output)
+		(at 220.98 186.69 180)
 		(fields_autoplaced yes)
 		(effects
@@
 		)
 		(property "Intersheetrefs" "${INTERSHEET_REFS}"
-			(at 138.2872 67.31 0)
+			(at 210.1934 186.69 0)
 			(effects
 				(font
@@
 		)
 	)
-	(global_label "PB4"
-		(shape bidirectional)
-		(at 375.92 195.58 0)
+	(global_label "3V3"
+		(shape input)
+		(at 144.78 67.31 180)
 		(fields_autoplaced yes)
 		(effects
@@
 				(size 1.27 1.27)
 			)
-			(justify left)
+			(justify right)
 		)
 		(property "Intersheetrefs" "${INTERSHEET_REFS}"
-			(at 383.766 195.58 0)
+			(at 138.2872 67.31 0)
 			(effects
 				(font
 					(size 1.27 1.27)
 				)
-				(justify left)
+				(justify right)
 				(hide yes)
 			)
@@
 			)
 		)
-		(property "Footprint" "Capacitor_SMD:C_0603_1608Metric_Pad1.08x0.95mm_HandSolder"
+		(property "Footprint" "Capacitor_SMD:C_0805_2012Metric_Pad1.18x1.45mm_HandSolder"
 			(at 151.4348 154.94 0)
 			(effects
@@
 			)
 		)
-		(property "Footprint" "Capacitor_SMD:C_0603_1608Metric_Pad1.08x0.95mm_HandSolder"
+		(property "Footprint" "Capacitor_SMD:C_0805_2012Metric_Pad1.18x1.45mm_HandSolder"
 			(at 166.0652 162.56 0)
 			(effects
@@
 			)
 		)
-		(property "Footprint" "Button_Switch_SMD:SW_Tactile_SPST_NO_Straight_CK_PTS636Sx25SMTRLFS"
+		(property "Footprint" "Button_Switch_SMD:SW_Push_1P1T_NO_CK_KMR2"
 			(at 158.75 59.69 0)
 			(effects
